Commit message: Updates to demo code.

File: models/pizza_cutter/pizza_cutter.urdf (robot description, URDF)
Before this commit: robot pizza_cutter, 1 links, 0 joints
Links:
- link pizza_cutter: mass None -> 0.02; geometry collision box size=0.0001 0.0001 0.0001; visual mesh filename=package://pizza_demo/models/pizza_cutter/meshes/pizza_cutte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

File: models/pizza_plate/pizza_plate.urdf (robot description, URDF)
Before this commit: robot pizza_plate, 1 links, 0 joints
Links:
- link pizza_plate: mass None -> 0.02; geometry collision box size=0.0001 0.0001 0.0001; visual mesh filename=package://pizza_demo/models/pizza_plate/meshes/pizza_plate_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
