Commit message: Trying to make the robot less colorful.

File: models/altered_pr2/gripper.urdf.xacro (robot description, xacro)
@@ -118,5 +118,5 @@
           <mesh filename="package://pr2_description/meshes/gripper_v0/l_finger_tip.dae" />
         </geometry>
-        <material name="Green" />
+        <material name="Grey" /> <!-- Green -->
       </visual>
       <collision>
@@ -150,5 +150,5 @@
           <mesh filename="package://pr2_description/meshes/gripper_v0/l_finger_tip.dae"  />
         </geometry>
-        <material name="Green" />
+        <material name="Grey" /> <!-- Green -->
       </visual>
       <collision>
@@ -181,5 +181,5 @@
           <mesh filename="package://pr2_description/meshes/gripper_v0/gripper_palm.dae"  />
         </geometry>
-        <material name="Red" />
+        <material name="Grey" /> <!-- Red -->
       </visual>
       <collision>
